File: kids-control-panel/kids-control-panel.kicad_pcb (KiCad board)
At the start: 2 copper layers, 4 parts, among them U1 CA56-12SURKWA, U2 MCP23017_SP Expander Module, U3 TFT LCD

Commit message: cad file changes
Other:
- board outline added: 68 x 65 mm
Changed lines of the file:
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@@
     )
   )
+  (gr_line (start -46.385 -88.576) (end -38.685 -88.576) (angle 90) (layer Edge.Cuts) (width 0.05))
+  (gr_line (start -38.685 -88.576) (end -38.685 -85.576) (angle 90) (layer Edge.Cuts) (width 0.05))
+  (gr_line (start -38.685 -85.576) (end -46.385 -85.576) (angle 90) (layer Edge.Cuts) (width 0.05))
+  (gr_line (start -46.385 -85.576) (end -46.385 -88.576) (angle 90) (layer Edge.Cuts) (width 0.05))
+  (gr_line (start -33.815 -88.578) (end -26.115 -88.578) (angle 90) (layer Edge.Cuts) (width 0.05))
+  (gr_line (start -26.115 -88.578) (end -26.115 -85.578) (angle 90) (layer Edge.Cuts) (width 0.05))
+  (gr_line (start -26.115 -85.578) (end -33.815 -85.578) (angle 90) (layer Edge.Cuts) (width 0.05))
+  (gr_line (start -33.815 -85.578) (end -33.815 -88.578) (angle 90) (layer Edge.Cuts) (width 0.05))
+  (gr_line (start -21.245 -88.579) (end -13.545 -88.579) (angle 90) (layer Edge.Cuts) (width 0.05))
+  (gr_line (start -13.545 -88.579) (end -13.545 -85.579) (angle 90) (layer Edge.Cuts) (width 0.05))
+  (gr_line (start -13.545 -85.579) (end -21.245 -85.579) (angle 90) (layer Edge.Cuts) (width 0.05))
+  (gr_line (start -21.245 -85.579) (end -21.245 -88.579) (angle 90) (layer Edge.Cuts) (width 0.05))
+  (gr_line (start -8.675 -88.581) (end -0.975 -88.581) (angle 90) (layer Edge.Cuts) (width 0.05))
+  (gr_line (start -0.975 -88.581) (end -0.975 -85.581) (angle 90) (layer Edge.Cuts) (width 0.05))
+  (gr_line (start -0.975 -85.581) (end -8.675 -85.581) (angle 90) (layer Edge.Cuts) (width 0.05))
+  (gr_line (start -8.675 -85.581) (end -8.675 -88.581) (angle 90) (layer Edge.Cuts) (width 0.05))
+  (gr_line (start -51.204 -70.998) (end 3.796 -70.998) (angle 90) (layer Edge.Cuts) (width 0.05))
+  (gr_line (start 3.796 -70.998) (end 3.796 -67.998) (angle 90) (layer Edge.Cuts) (width 0.05))
+  (gr_line (start 3.796 -67.998) (end -51.204 -67.998) (angle 90) (layer Edge.Cuts) (width 0.05))
+  (gr_line (start -51.204 -67.998) (end -51.204 -70.998) (angle 90) (layer Edge.Cuts) (width 0.05))
+  (gr_line (start -48.302 -60.289) (end 1.698 -60.289) (angle 90) (layer Edge.Cuts) (width 0.05))
+  (gr_line (start 1.698 -60.289) (end 1.698 -41.289) (angle 90) (layer Edge.Cuts) (width 0.05))
+  (gr_line (start 1.698 -41.289) (end -48.302 -41.289) (angle 90) (layer Edge.Cuts) (width 0.05))
+  (gr_line (start -48.302 -41.289) (end -48.302 -60.289) (angle 90) (layer Edge.Cuts) (width 0.05))
+  (gr_line (start -57.000 -98.000) (end 11.000 -98.000) (angle 90) (layer Edge.Cuts) (width 0.05))
+  (gr_line (start 11.000 -98.000) (end 11.000 -33.000) (angle 90) (layer Edge.Cuts) (width 0.05))
+  (gr_line (start 11.000 -33.000) (end -57.000 -33.000) (angle 90) (layer Edge.Cuts) (width 0.05))
+  (gr_line (start -57.000 -33.000) (end -57.000 -98.000) (angle 90) (layer Edge.Cuts) (width 0.05))
+  (gr_circle (center 8.458 -35.475) (end 7.708 -35.475) (layer Edge.Cuts) (width 0.05))
+  (gr_circle (center -54.542 -35.421) (end -55.292 -35.421) (layer Edge.Cuts) (width 0.05))
+  (gr_circle (center 8.406 -95.475) (end 7.656 -95.475) (layer Edge.Cuts) (width 0.05))
+  (gr_circle (center -54.594 -95.421) (end -55.344 -95.421) (layer Edge.Cuts) (width 0.05))
 )
