File: cad/kids-control-panel/kids-control-panel.sch (KiCad schematic (older format))
At the start: 19 parts, among them SW1 TACT-SWITCH, SW2 TACT-SWITCH, SW3 TACT-SWITCH, SW4 TACT-SWITCH, SW5 KY-040, SW6 SW_SPST_LED, SW7 SW_SPST_LED, SW8 SW_SPST_LED, SW9 SW_SPST_LED, U1 MCP23017_SP Expander Module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

Commit message: Directory structure cleanup
Changed lines of the file:
@@
 $Descr A4 11693 8268
 encoding utf-8
-Sheet 1 2
+Sheet 1 3
 Title ""
 Date ""
@@
 Text GLabel 4000 1450 3    50   BiDi ~ 0
 I2C
-Wire Wire Line
-	1850 1350 1750 1350
-Wire Wire Line
-	1750 1350 1750 800
 Text GLabel 4400 1750 0    50   Output ~ 0
 EXP1_INTB
@@
 Wire Bus Line
 	5700 6600 5700 7350
+$Sheet
+S 5600 3800 900  800
+U 60804078
+F0 "Power Distribution" 50
+F1 "power-distrib.sch" 50
+$EndSheet
 $EndSCHEMATC
